Commit message: everything is working

File: test.urdf (robot description, URDF)
Before this commit: robot pepe, 15 links, 14 joints
Links:
- removed link 20
- removed link 41
- removed link 410
- removed link 44
- removed link 811
- removed link 812
- removed link 82
- removed link 83
- removed link 85
- removed link 86
- removed link 88
- removed link 89
- added link 0, mass 0.013122976984362541; collision cylinder length=0.05849309551434667 radius=0.2672322969443196; visual cylinder length=0.05849309551434667 radius=0.2672322969443196
- added link 21, mass 0.0718395673333176; collision cylinder length=0.16282648844208059 radius=0.3747523710002725; visual cylinder length=0.16282648844208059 radius=0.3747523710002725
- added link 412, mass 0.9133123144896862; collision cylinder length=0.6178750735279873 radius=0.6859372418117727; visual cylinder length=0.6178750735279873 radius=0.6859372418117727
- added link 417, mass 0.9133123144896862; collision cylinder length=0.6178750735279873 radius=0.6859372418117727; visual cylinder length=0.6178750735279873 radius=0.6859372418117727
- added link 42, mass 0.9133123144896862; collision cylinder length=0.6178750735279873 radius=0.6859372418117727; visual cylinder length=0.6178750735279873 radius=0.6859372418117727
- added link 610, mass 1.5866702387245637; collision cylinder length=0.866141299474304 radius=0.7636142564097401; visual cylinder length=0.866141299474304 radius=0.7636142564097401
- added link 611, mass 1.5866702387245637; collision cylinder length=0.866141299474304 radius=0.7636142564097401; visual cylinder length=0.866141299474304 radius=0.7636142564097401
- added link 615, mass 1.5866702387245637; collision cylinder length=0.866141299474304 radius=0.7636142564097401; visual cylinder length=0.866141299474304 radius=0.7636142564097401
- added link 616, mass 1.5866702387245637; collision cylinder length=0.866141299474304 radius=0.7636142564097401; visual cylinder length=0.866141299474304 radius=0.7636142564097401
- added link 618, mass 1.5866702387245637; collision cylinder length=0.866141299474304 radius=0.7636142564097401; visual cylinder length=0.866141299474304 radius=0.7636142564097401
- added link 619, mass 1.5866702387245637; collision cylinder length=0.866141299474304 radius=0.7636142564097401; visual cylinder length=0.866141299474304 radius=0.7636142564097401
- added link 620, mass 1.5866702387245637; collision cylinder length=0.866141299474304 radius=0.7636142564097401; visual cylinder length=0.866141299474304 radius=0.7636142564097401
- added link 621, mass 1.5866702387245637; collision cylinder length=0.866141299474304 radius=0.7636142564097401; visual cylinder length=0.866141299474304 radius=0.7636142564097401
- added link 63, mass 1.5866702387245637; collision cylinder length=0.866141299474304 radius=0.7636142564097401; visual cylinder length=0.866141299474304 radius=0.7636142564097401
- added link 64, mass 1.5866702387245637; collision cylinder length=0.866141299474304 radius=0.7636142564097401; visual cylinder length=0.866141299474304 radius=0.7636142564097401
- added link 65, mass 1.5866702387245637; collision cylinder length=0.866141299474304 radius=0.7636142564097401; visual cylinder length=0.866141299474304 radius=0.7636142564097401
- added link 66, mass 1.5866702387245637; collision cylinder length=0.866141299474304 radius=0.7636142564097401; visual cylinder length=0.866141299474304 radius=0.7636142564097401
- added link 68, mass 1.5866702387245637; collision cylinder length=0.866141299474304 radius=0.7636142564097401; visual cylinder length=0.866141299474304 radius=0.7636142564097401
- added link 69, mass 1.5866702387245637; collision cylinder length=0.866141299474304 radius=0.7636142564097401; visual cylinder length=0.866141299474304 radius=0.7636142564097401
- added link 822, mass 0.03304298386168493; collision cylinder length=0.2584379173334501 radius=0.20173747301759215; visual cylinder length=0.2584379173334501 radius=0.20173747301759215
- added link 823, mass 0.03304298386168493; collision cylinder length=0.2584379173334501 radius=0.20173747301759215; visual cylinder length=0.2584379173334501 radius=0.20173747301759215
- link 47: mass None -> 0.9133123144896862; geometry collision cylinder length=0.6178750735279873 radius=0.6859372418117727; visual cylinder length=0.6178750735279873 radius=0.6859372418117727
- link 613: mass None -> 1.5866702387245637; geometry collision cylinder length=0.866141299474304 radius=0.7636142564097401; visual cylinder length=0.866141299474304 radius=0.7636142564097401
- link 614: mass None -> 1.5866702387245637; geometry collision cylinder length=0.866141299474304 radius=0.7636142564097401; visual cylinder length=0.866141299474304 radius=0.7636142564097401
Joints:
- removed joint 410_to_0
- removed joint 41_to_0
- removed joint 44_to_0
- removed joint 47_to_0
- removed joint 613_to_0
- removed joint 614_to_0
- removed joint 811_to_410
- removed joint 812_to_410
- removed joint 82_to_41
- removed joint 83_to_41
- removed joint 85_to_44
- removed joint 86_to_44
- removed joint 88_to_47
- removed joint 89_to_47
- added joint 21_to_0: type revolute, parent 0, child 21, origin xyz=0.6153185535048875 0.8281195361186879 0.3191120758285021 rpy=4.737322119911407 6.124536302366743 4.782791001722313, axis 0 1 0, limit lower=1 upper=0 effort=1 velocity=1
- added joint 412_to_21: type revolute, parent 21, child 412, origin xyz=0.12969784598227296 0.27539110039487547 0.40671554970209556 rpy=0.018932065802115334 3.980159367506136 5.84698508674984, axis 1 0 0, limit lower=1 upper=0 effort=1 velocity=1
- added joint 417_to_21: type revolute, parent 21, child 417, origin xyz=0.12969784598227296 0.27539110039487547 0.40671554970209556 rpy=0.018932065802115334 3.980159367506136 5.84698508674984, axis 1 0 0, limit lower=1 upper=0 effort=1 velocity=1
- added joint 42_to_21: type revolute, parent 21, child 42, origin xyz=0.12969784598227296 0.27539110039487547 0.40671554970209556 rpy=0.018932065802115334 3.980159367506136 5.84698508674984, axis 1 0 0, limit lower=1 upper=0 effort=1 velocity=1
- added joint 47_to_21: type revolute, parent 21, child 47, origin xyz=0.12969784598227296 0.27539110039487547 0.40671554970209556 rpy=0.018932065802115334 3.980159367506136 5.84698508674984, axis 1 0 0, limit lower=1 upper=0 effort=1 velocity=1
- added joint 610_to_47: type revolute, parent 47, child 610, origin xyz=0.41116557929850117 0.20966104753986026 0.7284829723228076 rpy=5.986797651657427 5.735764077859907 1.8159829719941722, axis 0 0 1, limit lower=1 upper=0 effort=1 velocity=1
- added joint 611_to_47: type revolute, parent 47, child 611, origin xyz=0.41116557929850117 0.20966104753986026 0.7284829723228076 rpy=5.986797651657427 5.735764077859907 1.8159829719941722, axis 0 0 1, limit lower=1 upper=0 effort=1 velocity=1
- added joint 613_to_412: type revolute, parent 412, child 613, origin xyz=0.41116557929850117 0.20966104753986026 0.7284829723228076 rpy=5.986797651657427 5.735764077859907 1.8159829719941722, axis 0 0 1, limit lower=1 upper=0 effort=1 velocity=1
- added joint 614_to_412: type revolute, parent 412, child 614, origin xyz=0.41116557929850117 0.20966104753986026 0.7284829723228076 rpy=5.986797651657427 5.735764077859907 1.8159829719941722, axis 0 0 1, limit lower=1 upper=0 effort=1 velocity=1
- added joint 615_to_412: type revolute, parent 412, child 615, origin xyz=0.41116557929850117 0.20966104753986026 0.7284829723228076 rpy=5.986797651657427 5.735764077859907 1.8159829719941722, axis 0 0 1, limit lower=1 upper=0 effort=1 velocity=1
- added joint 616_to_412: type revolute, parent 412, child 616, origin xyz=0.41116557929850117 0.20966104753986026 0.7284829723228076 rpy=5.986797651657427 5.735764077859907 1.8159829719941722, axis 0 0 1, limit lower=1 upper=0 effort=1 velocity=1
- added joint 618_to_417: type revolute, parent 417, child 618, origin xyz=0.41116557929850117 0.20966104753986026 0.7284829723228076 rpy=5.986797651657427 5.735764077859907 1.8159829719941722, axis 0 0 1, limit lower=1 upper=0 effort=1 velocity=1
- added joint 619_to_417: type revolute, parent 417, child 619, origin xyz=0.41116557929850117 0.20966104753986026 0.7284829723228076 rpy=5.986797651657427 5.735764077859907 1.8159829719941722, axis 0 0 1, limit lower=1 upper=0 effort=1 velocity=1
- added joint 620_to_417: type revolute, parent 417, child 620, origin xyz=0.41116557929850117 0.20966104753986026 0.7284829723228076 rpy=5.986797651657427 5.735764077859907 1.8159829719941722, axis 0 0 1, limit lower=1 upper=0 effort=1 velocity=1
- added joint 621_to_417: type revolute, parent 417, child 621, origin xyz=0.41116557929850117 0.20966104753986026 0.7284829723228076 rpy=5.986797651657427 5.735764077859907 1.8159829719941722, axis 0 0 1, limit lower=1 upper=0 effort=1 velocity=1
- added joint 63_to_42: type revolute, parent 42, child 63, origin xyz=0.41116557929850117 0.20966104753986026 0.7284829723228076 rpy=5.986797651657427 5.735764077859907 1.8159829719941722, axis 0 0 1, limit lower=1 upper=0 effort=1 velocity=1
- added joint 64_to_42: type revolute, parent 42, child 64, origin xyz=0.41116557929850117 0.20966104753986026 0.7284829723228076 rpy=5.986797651657427 5.735764077859907 1.8159829719941722, axis 0 0 1, limit lower=1 upper=0 effort=1 velocity=1
- added joint 65_to_42: type revolute, parent 42, child 65, origin xyz=0.41116557929850117 0.20966104753986026 0.7284829723228076 rpy=5.986797651657427 5.735764077859907 1.8159829719941722, axis 0 0 1, limit lower=1 upper=0 effort=1 velocity=1
- added joint 66_to_42: type revolute, parent 42, child 66, origin xyz=0.41116557929850117 0.20966104753986026 0.7284829723228076 rpy=5.986797651657427 5.735764077859907 1.8159829719941722, axis 0 0 1, limit lower=1 upper=0 effort=1 velocity=1
- added joint 68_to_47: type revolute, parent 47, child 68, origin xyz=0.41116557929850117 0.20966104753986026 0.7284829723228076 rpy=5.986797651657427 5.735764077859907 1.8159829719941722, axis 0 0 1, limit lower=1 upper=0 effort=1 velocity=1
- added joint 69_to_47: type revolute, parent 47, child 69, origin xyz=0.41116557929850117 0.20966104753986026 0.7284829723228076 rpy=5.986797651657427 5.735764077859907 1.8159829719941722, axis 0 0 1, limit lower=1 upper=0 effort=1 velocity=1
- added joint 822_to_0: type revolute, parent 0, child 822, origin xyz=0.7342663889755077 0.7326829410186347 0.6227828917287632 rpy=2.4939088153879307 5.43482740156142 1.4288995407759828, axis 0 1 0, limit lower=1 upper=0 effort=1 velocity=1
- added joint 823_to_0: type revolute, parent 0, child 823, origin xyz=0.7342663889755077 0.7326829410186347 0.6227828917287632 rpy=2.4939088153879307 5.43482740156142 1.4288995407759828, axis 0 1 0, limit lower=1 upper=0 effort=1 velocity=1
