Commit message: edited gitignore

File: test.urdf (robot description, URDF)
Before this commit: robot pepe, 24 links, 23 joints
Links:
- removed link 412
- removed link 417
- removed link 613
- removed link 614
- removed link 615
- removed link 616
- removed link 621
- removed link 822
- removed link 823
- added link 215, mass 0.6524059645529954; collision cylinder length=0.6231442835960798 radius=0.5772842613810276; visual cylinder length=0.6231442835960798 radius=0.5772842613810276
- added link 416, mass 0.8325837026567471; collision cylinder length=0.36629808497581684 radius=0.8505927806729483; visual cylinder length=0.36629808497581684 radius=0.8505927806729483
- added link 421, mass 0.8325837026567471; collision cylinder length=0.36629808497581684 radius=0.8505927806729483; visual cylinder length=0.36629808497581684 radius=0.8505927806729483
- added link 617, mass 0.010832931136616195; collision cylinder length=0.2726205469266557 radius=0.11246535604554542; visual cylinder length=0.2726205469266557 radius=0.11246535604554542
- added link 622, mass 0.010832931136616195; collision cylinder length=0.2726205469266557 radius=0.11246535604554542; visual cylinder length=0.2726205469266557 radius=0.11246535604554542
- added link 623, mass 0.010832931136616195; collision cylinder length=0.2726205469266557 radius=0.11246535604554542; visual cylinder length=0.2726205469266557 radius=0.11246535604554542
- added link 624, mass 0.010832931136616195; collision cylinder length=0.2726205469266557 radius=0.11246535604554542; visual cylinder length=0.2726205469266557 radius=0.11246535604554542
- added link 625, mass 0.010832931136616195; collision cylinder length=0.2726205469266557 radius=0.11246535604554542; visual cylinder length=0.2726205469266557 radius=0.11246535604554542
- added link 812, mass 0.3389775328179271; collision cylinder length=0.3503023462419469 radius=0.5549949070504262; visual cylinder length=0.3503023462419469 radius=0.5549949070504262
- added link 813, mass 0.3389775328179271; collision cylinder length=0.3503023462419469 radius=0.5549949070504262; visual cylinder length=0.3503023462419469 radius=0.5549949070504262
- added link 814, mass 0.3389775328179271; collision cylinder length=0.3503023462419469 radius=0.5549949070504262; visual cylinder length=0.3503023462419469 radius=0.5549949070504262
- added link 826, mass 0.3389775328179271; collision cylinder length=0.3503023462419469 radius=0.5549949070504262; visual cylinder length=0.3503023462419469 radius=0.5549949070504262
- added link 827, mass 0.3389775328179271; collision cylinder length=0.3503023462419469 radius=0.5549949070504262; visual cylinder length=0.3503023462419469 radius=0.5549949070504262
- added link 828, mass 0.3389775328179271; collision cylinder length=0.3503023462419469 radius=0.5549949070504262; visual cylinder length=0.3503023462419469 radius=0.5549949070504262
- link 0: mass 0.013122976984362541 -> 0.28590603454908253; geometry collision cylinder length=0.4355018576387162 radius=0.45713210004498905; visual cylinder length=0.4355018576387162 radius=0.45713210004498905
- link 21: mass 0.0718395673333176 -> 0.6524059645529954; geometry collision cylinder length=0.6231442835960798 radius=0.5772842613810276; visual cylinder length=0.6231442835960798 radius=0.5772842613810276
- link 42: mass 0.9133123144896862 -> 0.8325837026567471; geometry collision cylinder length=0.36629808497581684 radius=0.8505927806729483; visual cylinder length=0.36629808497581684 radius=0.8505927806729483
- link 47: mass 0.9133123144896862 -> 0.8325837026567471; geometry collision cylinder length=0.36629808497581684 radius=0.8505927806729483; visual cylinder length=0.36629808497581684 radius=0.8505927806729483
- link 610: mass 1.5866702387245637 -> 0.010832931136616195; geometry collision cylinder length=0.2726205469266557 radius=0.11246535604554542; visual cylinder length=0.2726205469266557 radius=0.11246535604554542
- link 611: mass 1.5866702387245637 -> 0.010832931136616195; geometry collision cylinder length=0.2726205469266557 radius=0.11246535604554542; visual cylinder length=0.2726205469266557 radius=0.11246535604554542
- link 618: mass 1.5866702387245637 -> 0.010832931136616195; geometry collision cylinder length=0.2726205469266557 radius=0.11246535604554542; visual cylinder length=0.2726205469266557 radius=0.11246535604554542
- link 619: mass 1.5866702387245637 -> 0.010832931136616195; geometry collision cylinder length=0.2726205469266557 radius=0.11246535604554542; visual cylinder length=0.2726205469266557 radius=0.11246535604554542
- link 620: mass 1.5866702387245637 -> 0.010832931136616195; geometry collision cylinder length=0.2726205469266557 radius=0.11246535604554542; visual cylinder length=0.2726205469266557 radius=0.11246535604554542
- link 63: mass 1.5866702387245637 -> 0.010832931136616195; geometry collision cylinder length=0.2726205469266557 radius=0.11246535604554542; visual cylinder length=0.2726205469266557 radius=0.11246535604554542
- link 64: mass 1.5866702387245637 -> 0.010832931136616195; geometry collision cylinder length=0.2726205469266557 radius=0.11246535604554542; visual cylinder length=0.2726205469266557 radius=0.11246535604554542
- link 65: mass 1.5866702387245637 -> 0.010832931136616195; geometry collision cylinder length=0.2726205469266557 radius=0.11246535604554542; visual cylinder length=0.2726205469266557 radius=0.11246535604554542
- link 66: mass 1.5866702387245637 -> 0.010832931136616195; geometry collision cylinder length=0.2726205469266557 radius=0.11246535604554542; visual cylinder length=0.2726205469266557 radius=0.11246535604554542
- link 68: mass 1.5866702387245637 -> 0.010832931136616195; geometry collision cylinder length=0.2726205469266557 radius=0.11246535604554542; visual cylinder length=0.2726205469266557 radius=0.11246535604554542
- link 69: mass 1.5866702387245637 -> 0.010832931136616195; geometry collision cylinder length=0.2726205469266557 radius=0.11246535604554542; visual cylinder length=0.2726205469266557 radius=0.11246535604554542
Joints:
- removed joint 412_to_21
- removed joint 417_to_21
- removed joint 613_to_412
- removed joint 614_to_412
- removed joint 615_to_412
- removed joint 616_to_412
- removed joint 618_to_417
- removed joint 619_to_417
- removed joint 620_to_417
- removed joint 621_to_417
- removed joint 822_to_0
- removed joint 823_to_0
- added joint 215_to_0: type revolute, parent 0, child 215, origin xyz=0.19259146267304128 0.4917130192012905 0.349595212216125 rpy=5.456818844119362 1.060263834673811 0.7049385657791664, axis 1 0 0, limit lower=1 upper=0 effort=1 velocity=1
- added joint 416_to_215: type revolute, parent 215, child 416, origin xyz=0.6062801905323048 0.3688255471797607 0.38435090481182244 rpy=4.672786196184905 5.840986373449584 3.9807594868635974, axis 0 1 0, limit lower=1 upper=0 effort=1 velocity=1
- added joint 421_to_215: type revolute, parent 215, child 421, origin xyz=0.6062801905323048 0.3688255471797607 0.38435090481182244 rpy=4.672786196184905 5.840986373449584 3.9807594868635974, axis 0 1 0, limit lower=1 upper=0 effort=1 velocity=1
- added joint 617_to_416: type revolute, parent 416, child 617, origin xyz=0.21539652377926988 0.580339699481914 0.08187044449670677 rpy=4.810082160613909 5.4325319233382325 1.7369200020373337, axis 1 0 0, limit lower=1 upper=0 effort=1 velocity=1
- added joint 618_to_416: type revolute, parent 416, child 618, origin xyz=0.21539652377926988 0.580339699481914 0.08187044449670677 rpy=4.810082160613909 5.4325319233382325 1.7369200020373337, axis 1 0 0, limit lower=1 upper=0 effort=1 velocity=1
- added joint 619_to_416: type revolute, parent 416, child 619, origin xyz=0.21539652377926988 0.580339699481914 0.08187044449670677 rpy=4.810082160613909 5.4325319233382325 1.7369200020373337, axis 1 0 0, limit lower=1 upper=0 effort=1 velocity=1
- added joint 620_to_416: type revolute, parent 416, child 620, origin xyz=0.21539652377926988 0.580339699481914 0.08187044449670677 rpy=4.810082160613909 5.4325319233382325 1.7369200020373337, axis 1 0 0, limit lower=1 upper=0 effort=1 velocity=1
- added joint 622_to_421: type revolute, parent 421, child 622, origin xyz=0.21539652377926988 0.580339699481914 0.08187044449670677 rpy=4.810082160613909 5.4325319233382325 1.7369200020373337, axis 1 0 0, limit lower=1 upper=0 effort=1 velocity=1
- added joint 623_to_421: type revolute, parent 421, child 623, origin xyz=0.21539652377926988 0.580339699481914 0.08187044449670677 rpy=4.810082160613909 5.4325319233382325 1.7369200020373337, axis 1 0 0, limit lower=1 upper=0 effort=1 velocity=1
- added joint 624_to_421: type revolute, parent 421, child 624, origin xyz=0.21539652377926988 0.580339699481914 0.08187044449670677 rpy=4.810082160613909 5.4325319233382325 1.7369200020373337, axis 1 0 0, limit lower=1 upper=0 effort=1 velocity=1
- added joint 625_to_421: type revolute, parent 421, child 625, origin xyz=0.21539652377926988 0.580339699481914 0.08187044449670677 rpy=4.810082160613909 5.4325319233382325 1.7369200020373337, axis 1 0 0, limit lower=1 upper=0 effort=1 velocity=1
- added joint 812_to_21: type fixed, parent 21, child 812, origin xyz=0.5153052598637617 0.38110823267094396 0.08377386454918168 rpy=0.02430995934889007 0.033060986770781904 1.9778230288453595, axis 0 1 0, limit lower=1 upper=0 effort=1 velocity=1
- added joint 813_to_21: type fixed, parent 21, child 813, origin xyz=0.5153052598637617 0.38110823267094396 0.08377386454918168 rpy=0.02430995934889007 0.033060986770781904 1.9778230288453595, axis 0 1 0, limit lower=1 upper=0 effort=1 velocity=1
- added joint 814_to_21: type fixed, parent 21, child 814, origin xyz=0.5153052598637617 0.38110823267094396 0.08377386454918168 rpy=0.02430995934889007 0.033060986770781904 1.9778230288453595, axis 0 1 0, limit lower=1 upper=0 effort=1 velocity=1
- added joint 826_to_215: type fixed, parent 215, child 826, origin xyz=0.5153052598637617 0.38110823267094396 0.08377386454918168 rpy=0.02430995934889007 0.033060986770781904 1.9778230288453595, axis 0 1 0, limit lower=1 upper=0 effort=1 velocity=1
- added joint 827_to_215: type fixed, parent 215, child 827, origin xyz=0.5153052598637617 0.38110823267094396 0.08377386454918168 rpy=0.02430995934889007 0.033060986770781904 1.9778230288453595, axis 0 1 0, limit lower=1 upper=0 effort=1 velocity=1
- added joint 828_to_215: type fixed, parent 215, child 828, origin xyz=0.5153052598637617 0.38110823267094396 0.08377386454918168 rpy=0.02430995934889007 0.033060986770781904 1.9778230288453595, axis 0 1 0, limit lower=1 upper=0 effort=1 velocity=1
- joint 21_to_0: axis 0 1 0 -> 1 0 0; origin xyz=0.6153185535048875 0.8281195361186879 0.3191120758285021 rpy=4.737322119911407 6.124536302366743 4.782791001722313 -> xyz=0.19259146267304128 0.4917130192012905 0.349595212216125 rpy=5.456818844119362 1.060263834673811 0.7049385657791664
- joint 42_to_21: axis 1 0 0 -> 0 1 0; origin xyz=0.12969784598227296 0.27539110039487547 0.40671554970209556 rpy=0.018932065802115334 3.980159367506136 5.84698508674984 -> xyz=0.6062801905323048 0.3688255471797607 0.38435090481182244 rpy=4.672786196184905 5.840986373449584 3.9807594868635974
- joint 47_to_21: axis 1 0 0 -> 0 1 0; origin xyz=0.12969784598227296 0.27539110039487547 0.40671554970209556 rpy=0.018932065802115334 3.980159367506136 5.84698508674984 -> xyz=0.6062801905323048 0.3688255471797607 0.38435090481182244 rpy=4.672786196184905 5.840986373449584 3.9807594868635974
- joint 610_to_47: axis 0 0 1 -> 1 0 0; origin xyz=0.41116557929850117 0.20966104753986026 0.7284829723228076 rpy=5.986797651657427 5.735764077859907 1.8159829719941722 -> xyz=0.21539652377926988 0.580339699481914 0.08187044449670677 rpy=4.810082160613909 5.4325319233382325 1.7369200020373337
- joint 611_to_47: axis 0 0 1 -> 1 0 0; origin xyz=0.41116557929850117 0.20966104753986026 0.7284829723228076 rpy=5.986797651657427 5.735764077859907 1.8159829719941722 -> xyz=0.21539652377926988 0.580339699481914 0.08187044449670677 rpy=4.810082160613909 5.4325319233382325 1.7369200020373337
- joint 63_to_42: axis 0 0 1 -> 1 0 0; origin xyz=0.41116557929850117 0.20966104753986026 0.7284829723228076 rpy=5.986797651657427 5.735764077859907 1.8159829719941722 -> xyz=0.21539652377926988 0.580339699481914 0.08187044449670677 rpy=4.810082160613909 5.4325319233382325 1.7369200020373337
- joint 64_to_42: axis 0 0 1 -> 1 0 0; origin xyz=0.41116557929850117 0.20966104753986026 0.7284829723228076 rpy=5.986797651657427 5.735764077859907 1.8159829719941722 -> xyz=0.21539652377926988 0.580339699481914 0.08187044449670677 rpy=4.810082160613909 5.4325319233382325 1.7369200020373337
- joint 65_to_42: axis 0 0 1 -> 1 0 0; origin xyz=0.41116557929850117 0.20966104753986026 0.7284829723228076 rpy=5.986797651657427 5.735764077859907 1.8159829719941722 -> xyz=0.21539652377926988 0.580339699481914 0.08187044449670677 rpy=4.810082160613909 5.4325319233382325 1.7369200020373337
- joint 66_to_42: axis 0 0 1 -> 1 0 0; origin xyz=0.41116557929850117 0.20966104753986026 0.7284829723228076 rpy=5.986797651657427 5.735764077859907 1.8159829719941722 -> xyz=0.21539652377926988 0.580339699481914 0.08187044449670677 rpy=4.810082160613909 5.4325319233382325 1.7369200020373337
- joint 68_to_47: axis 0 0 1 -> 1 0 0; origin xyz=0.41116557929850117 0.20966104753986026 0.7284829723228076 rpy=5.986797651657427 5.735764077859907 1.8159829719941722 -> xyz=0.21539652377926988 0.580339699481914 0.08187044449670677 rpy=4.810082160613909 5.4325319233382325 1.7369200020373337
- joint 69_to_47: axis 0 0 1 -> 1 0 0; origin xyz=0.41116557929850117 0.20966104753986026 0.7284829723228076 rpy=5.986797651657427 5.735764077859907 1.8159829719941722 -> xyz=0.21539652377926988 0.580339699481914 0.08187044449670677 rpy=4.810082160613909 5.4325319233382325 1.7369200020373337

Commit message: adding motors

File: test.urdf (robot description, URDF)
Before this commit: robot pepe, 29 links, 28 joints
Links:
- removed link 215
- removed link 416
- removed link 421
- removed link 47
- removed link 610
- removed link 611
- removed link 617
- removed link 618
- removed link 619
- removed link 620
- removed link 622
- removed link 623
- removed link 624
- removed link 625
- removed link 66
- removed link 812
- removed link 813
- removed link 814
- removed link 826
- removed link 827
- removed link 828
- added link 46, mass 0.1654554748651725; collision cylinder length=0.38405556734331214 radius=0.3703126963433502; visual cylinder length=0.38405556734331214 radius=0.3703126963433502
- added link 67, mass 0.050611127966738306; collision cylinder length=0.1023435365543045 radius=0.39675084627190904; visual cylinder length=0.1023435365543045 radius=0.39675084627190904
- link 0: mass 0.28590603454908253 -> 0.07203475117296865; geometry collision cylinder length=0.7440047389120009 radius=0.17555299493693666; visual cylinder length=0.7440047389120009 radius=0.17555299493693666
- link 21: mass 0.6524059645529954 -> 0.08887827174730793; geometry collision cylinder length=0.08179341151604225 radius=0.588116958986316; visual cylinder length=0.08179341151604225 radius=0.588116958986316
- link 42: mass 0.8325837026567471 -> 0.1654554748651725; geometry collision cylinder length=0.38405556734331214 radius=0.3703126963433502; visual cylinder length=0.38405556734331214 radius=0.3703126963433502
- link 63: mass 0.010832931136616195 -> 0.050611127966738306; geometry collision cylinder length=0.1023435365543045 radius=0.39675084627190904; visual cylinder length=0.1023435365543045 radius=0.39675084627190904
- link 64: mass 0.010832931136616195 -> 0.050611127966738306; geometry collision cylinder length=0.1023435365543045 radius=0.39675084627190904; visual cylinder length=0.1023435365543045 radius=0.39675084627190904
- link 65: mass 0.010832931136616195 -> 0.050611127966738306; geometry collision cylinder length=0.1023435365543045 radius=0.39675084627190904; visual cylinder length=0.1023435365543045 radius=0.39675084627190904
- link 68: mass 0.010832931136616195 -> 0.050611127966738306; geometry collision cylinder length=0.1023435365543045 radius=0.39675084627190904; visual cylinder length=0.1023435365543045 radius=0.39675084627190904
- link 69: mass 0.010832931136616195 -> 0.050611127966738306; geometry collision cylinder length=0.1023435365543045 radius=0.39675084627190904; visual cylinder length=0.1023435365543045 radius=0.39675084627190904
Joints:
- removed joint 215_to_0
- removed joint 416_to_215
- removed joint 421_to_215
- removed joint 47_to_21
- removed joint 610_to_47
- removed joint 611_to_47
- removed joint 617_to_416
- removed joint 618_to_416
- removed joint 619_to_416
- removed joint 620_to_416
- removed joint 622_to_421
- removed joint 623_to_421
- removed joint 624_to_421
- removed joint 625_to_421
- removed joint 66_to_42
- removed joint 68_to_47
- removed joint 69_to_47
- removed joint 812_to_21
- removed joint 813_to_21
- removed joint 814_to_21
- removed joint 826_to_215
- removed joint 827_to_215
- removed joint 828_to_215
- added joint 46_to_21: type revolute, parent 21, child 46, origin xyz=0.3435771423881663 0.873089580961556 0.5132473338229839 rpy=18.660283265952998 0.7667402962159244 5.87587692316254, axis 0 0 1, limit lower=1 upper=0 effort=1 velocity=1
- added joint 67_to_46: type fixed, parent 46, child 67, origin xyz=0.3303617565007204 0.27459723831782246 0.6819876324854989 rpy=8.2615093030568 5.452041652722386 0.33001066787858613, axis 0 0 1, limit lower=1 upper=0 effort=1 velocity=1
- added joint 68_to_46: type fixed, parent 46, child 68, origin xyz=0.3303617565007204 0.27459723831782246 0.6819876324854989 rpy=12.3922639545852 5.452041652722386 0.33001066787858613, axis 0 0 1, limit lower=1 upper=0 effort=1 velocity=1
- added joint 69_to_46: type fixed, parent 46, child 69, origin xyz=0.3303617565007204 0.27459723831782246 0.6819876324854989 rpy=16.5230186061136 5.452041652722386 0.33001066787858613, axis 0 0 1, limit lower=1 upper=0 effort=1 velocity=1
- joint 21_to_0: axis 1 0 0 -> 0 1 0; origin xyz=0.19259146267304128 0.4917130192012905 0.349595212216125 rpy=5.456818844119362 1.060263834673811 0.7049385657791664 -> xyz=0.25178959442183646 0.5180386228097638 0.6914972374434389 rpy=1.653386999011431 4.9916447991114845 3.763602437403395
- joint 42_to_21: axis 0 1 0 -> 0 0 1; origin xyz=0.6062801905323048 0.3688255471797607 0.38435090481182244 rpy=4.672786196184905 5.840986373449584 3.9807594868635974 -> xyz=0.3435771423881663 0.873089580961556 0.5132473338229839 rpy=12.440188843968665 0.7667402962159244 5.87587692316254
- joint 63_to_42: axis 1 0 0 -> 0 0 1; origin xyz=0.21539652377926988 0.580339699481914 0.08187044449670677 rpy=4.810082160613909 5.4325319233382325 1.7369200020373337 -> xyz=0.3303617565007204 0.27459723831782246 0.6819876324854989 rpy=8.2615093030568 5.452041652722386 0.33001066787858613; type revolute -> fixed
- joint 64_to_42: axis 1 0 0 -> 0 0 1; origin xyz=0.21539652377926988 0.580339699481914 0.08187044449670677 rpy=4.810082160613909 5.4325319233382325 1.7369200020373337 -> xyz=0.3303617565007204 0.27459723831782246 0.6819876324854989 rpy=12.3922639545852 5.452041652722386 0.33001066787858613; type revolute -> fixed
- joint 65_to_42: axis 1 0 0 -> 0 0 1; origin xyz=0.21539652377926988 0.580339699481914 0.08187044449670677 rpy=4.810082160613909 5.4325319233382325 1.7369200020373337 -> xyz=0.3303617565007204 0.27459723831782246 0.6819876324854989 rpy=16.5230186061136 5.452041652722386 0.33001066787858613; type revolute -> fixed
