Commit message: fixed some issues

File: test.urdf (robot description, URDF)
Before this commit: robot pepe, 10 links, 9 joints
Links:
- removed link 46
- removed link 67
- added link 412, mass 0.06597561133511197; collision cylinder length=0.40479181187133173 radius=0.2277723044407879; visual cylinder length=0.40479181187133173 radius=0.2277723044407879
- added link 47, mass 0.06597561133511197; collision cylinder length=0.40479181187133173 radius=0.2277723044407879; visual cylinder length=0.40479181187133173 radius=0.2277723044407879
- added link 610, mass 0.22329004334489153; collision cylinder length=0.254929525917195 radius=0.5280191498122452; visual cylinder length=0.254929525917195 radius=0.5280191498122452
- added link 611, mass 0.22329004334489153; collision cylinder length=0.254929525917195 radius=0.5280191498122452; visual cylinder length=0.254929525917195 radius=0.5280191498122452
- added link 613, mass 0.22329004334489153; collision cylinder length=0.254929525917195 radius=0.5280191498122452; visual cylinder length=0.254929525917195 radius=0.5280191498122452
- added link 614, mass 0.22329004334489153; collision cylinder length=0.254929525917195 radius=0.5280191498122452; visual cylinder length=0.254929525917195 radius=0.5280191498122452
- added link 615, mass 0.22329004334489153; collision cylinder length=0.254929525917195 radius=0.5280191498122452; visual cylinder length=0.254929525917195 radius=0.5280191498122452
- added link 616, mass 0.22329004334489153; collision cylinder length=0.254929525917195 radius=0.5280191498122452; visual cylinder length=0.254929525917195 radius=0.5280191498122452
- added link 66, mass 0.22329004334489153; collision cylinder length=0.254929525917195 radius=0.5280191498122452; visual cylinder length=0.254929525917195 radius=0.5280191498122452
- added link 817, mass 1.2162402138230586; collision cylinder length=0.8880666198940113 radius=0.6602554122427263; visual cylinder length=0.8880666198940113 radius=0.6602554122427263
- added link 818, mass 1.2162402138230586; collision cylinder length=0.8880666198940113 radius=0.6602554122427263; visual cylinder length=0.8880666198940113 radius=0.6602554122427263
- added link 819, mass 1.2162402138230586; collision cylinder length=0.8880666198940113 radius=0.6602554122427263; visual cylinder length=0.8880666198940113 radius=0.6602554122427263
- added link 820, mass 1.2162402138230586; collision cylinder length=0.8880666198940113 radius=0.6602554122427263; visual cylinder length=0.8880666198940113 radius=0.6602554122427263
- link 0: mass 0.07203475117296865 -> 0.48167678407889525; geometry collision cylinder length=0.5613390321358644 radius=0.5226251440050671; visual cylinder length=0.5613390321358644 radius=0.5226251440050671
- link 21: mass 0.08887827174730793 -> 0.3517009485578119; geometry collision cylinder length=0.4754698360498949 radius=0.4852330216088294; visual cylinder length=0.4754698360498949 radius=0.4852330216088294
- link 42: mass 0.1654554748651725 -> 0.06597561133511197; geometry collision cylinder length=0.40479181187133173 radius=0.2277723044407879; visual cylinder length=0.40479181187133173 radius=0.2277723044407879
- link 63: mass 0.050611127966738306 -> 0.22329004334489153; geometry collision cylinder length=0.254929525917195 radius=0.5280191498122452; visual cylinder length=0.254929525917195 radius=0.5280191498122452
- link 64: mass 0.050611127966738306 -> 0.22329004334489153; geometry collision cylinder length=0.254929525917195 radius=0.5280191498122452; visual cylinder length=0.254929525917195 radius=0.5280191498122452
- link 65: mass 0.050611127966738306 -> 0.22329004334489153; geometry collision cylinder length=0.254929525917195 radius=0.5280191498122452; visual cylinder length=0.254929525917195 radius=0.5280191498122452
- link 68: mass 0.050611127966738306 -> 0.22329004334489153; geometry collision cylinder length=0.254929525917195 radius=0.5280191498122452; visual cylinder length=0.254929525917195 radius=0.5280191498122452
- link 69: mass 0.050611127966738306 -> 0.22329004334489153; geometry collision cylinder length=0.254929525917195 radius=0.5280191498122452; visual cylinder length=0.254929525917195 radius=0.5280191498122452
Joints:
- removed joint 42_to_21
- removed joint 46_to_21
- removed joint 67_to_46
- removed joint 68_to_46
- removed joint 69_to_46
- added joint 412_to_0: type revolute, parent 0, child 412, origin xyz=0.7305803756326614 0.9597435036802869 0.5691345814086761 rpy=20.251409588401224 2.7081443593182803 1.7607576692902518, axis 0 0 1, limit lower=1 upper=0 effort=1 velocity=1
- added joint 42_to_0: type revolute, parent 0, child 42, origin xyz=0.7305803756326614 0.9597435036802869 0.5691345814086761 rpy=12.150845753040734 2.7081443593182803 1.7607576692902518, axis 0 0 1, limit lower=1 upper=0 effort=1 velocity=1
- added joint 47_to_0: type revolute, parent 0, child 47, origin xyz=0.7305803756326614 0.9597435036802869 0.5691345814086761 rpy=16.20112767072098 2.7081443593182803 1.7607576692902518, axis 0 0 1, limit lower=1 upper=0 effort=1 velocity=1
- added joint 610_to_47: type revolute, parent 47, child 610, origin xyz=0.49248509879307456 0.5384094529224637 0.47381226345960226 rpy=7.113604658193993 6.186895727104294 1.21732181032596, axis 0 1 0, limit lower=1 upper=0 effort=1 velocity=1
- added joint 611_to_47: type revolute, parent 47, child 611, origin xyz=0.49248509879307456 0.5384094529224637 0.47381226345960226 rpy=8.892005822742492 6.186895727104294 1.21732181032596, axis 0 1 0, limit lower=1 upper=0 effort=1 velocity=1
- added joint 613_to_412: type revolute, parent 412, child 613, origin xyz=0.49248509879307456 0.5384094529224637 0.47381226345960226 rpy=3.5568023290969966 6.186895727104294 1.21732181032596, axis 0 1 0, limit lower=1 upper=0 effort=1 velocity=1
- added joint 614_to_412: type revolute, parent 412, child 614, origin xyz=0.49248509879307456 0.5384094529224637 0.47381226345960226 rpy=5.335203493645495 6.186895727104294 1.21732181032596, axis 0 1 0, limit lower=1 upper=0 effort=1 velocity=1
- added joint 615_to_412: type revolute, parent 412, child 615, origin xyz=0.49248509879307456 0.5384094529224637 0.47381226345960226 rpy=7.113604658193993 6.186895727104294 1.21732181032596, axis 0 1 0, limit lower=1 upper=0 effort=1 velocity=1
- added joint 616_to_412: type revolute, parent 412, child 616, origin xyz=0.49248509879307456 0.5384094529224637 0.47381226345960226 rpy=8.892005822742492 6.186895727104294 1.21732181032596, axis 0 1 0, limit lower=1 upper=0 effort=1 velocity=1
- added joint 66_to_42: type revolute, parent 42, child 66, origin xyz=0.49248509879307456 0.5384094529224637 0.47381226345960226 rpy=8.892005822742492 6.186895727104294 1.21732181032596, axis 0 1 0, limit lower=1 upper=0 effort=1 velocity=1
- added joint 68_to_47: type revolute, parent 47, child 68, origin xyz=0.49248509879307456 0.5384094529224637 0.47381226345960226 rpy=3.5568023290969966 6.186895727104294 1.21732181032596, axis 0 1 0, limit lower=1 upper=0 effort=1 velocity=1
- added joint 69_to_47: type revolute, parent 47, child 69, origin xyz=0.49248509879307456 0.5384094529224637 0.47381226345960226 rpy=5.335203493645495 6.186895727104294 1.21732181032596, axis 0 1 0, limit lower=1 upper=0 effort=1 velocity=1
- added joint 817_to_0: type fixed, parent 0, child 817, origin xyz=0.28971721708000076 0.5584616802894801 0.07583618472640796 rpy=32.84915237089584 4.277521008339037 1.3580870259551947, axis 0 1 0, limit lower=1 upper=0 effort=1 velocity=1
- added joint 818_to_0: type fixed, parent 0, child 818, origin xyz=0.28971721708000076 0.5584616802894801 0.07583618472640796 rpy=38.324011099378474 4.277521008339037 1.3580870259551947, axis 0 1 0, limit lower=1 upper=0 effort=1 velocity=1
- added joint 819_to_0: type fixed, parent 0, child 819, origin xyz=0.28971721708000076 0.5584616802894801 0.07583618472640796 rpy=43.79886982786111 4.277521008339037 1.3580870259551947, axis 0 1 0, limit lower=1 upper=0 effort=1 velocity=1
- added joint 820_to_0: type fixed, parent 0, child 820, origin xyz=0.28971721708000076 0.5584616802894801 0.07583618472640796 rpy=49.27372855634375 4.277521008339037 1.3580870259551947, axis 0 1 0, limit lower=1 upper=0 effort=1 velocity=1
- joint 21_to_0: axis 0 1 0 -> 0 0 1; origin xyz=0.25178959442183646 0.5180386228097638 0.6914972374434389 rpy=1.653386999011431 4.9916447991114845 3.763602437403395 -> xyz=0.4049974900486498 0.29998392026674536 0.7898189595844443 rpy=2.882601938893883 3.9758946769399803 1.974408129937515; type revolute -> fixed
- joint 63_to_42: axis 0 0 1 -> 0 1 0; origin xyz=0.3303617565007204 0.27459723831782246 0.6819876324854989 rpy=8.2615093030568 5.452041652722386 0.33001066787858613 -> xyz=0.49248509879307456 0.5384094529224637 0.47381226345960226 rpy=3.5568023290969966 6.186895727104294 1.21732181032596; type fixed -> revolute
- joint 64_to_42: axis 0 0 1 -> 0 1 0; origin xyz=0.3303617565007204 0.27459723831782246 0.6819876324854989 rpy=12.3922639545852 5.452041652722386 0.33001066787858613 -> xyz=0.49248509879307456 0.5384094529224637 0.47381226345960226 rpy=5.335203493645495 6.186895727104294 1.21732181032596; type fixed -> revolute
- joint 65_to_42: axis 0 0 1 -> 0 1 0; origin xyz=0.3303617565007204 0.27459723831782246 0.6819876324854989 rpy=16.5230186061136 5.452041652722386 0.33001066787858613 -> xyz=0.49248509879307456 0.5384094529224637 0.47381226345960226 rpy=7.113604658193993 6.186895727104294 1.21732181032596; type fixed -> revolute
