Commit message: implement fitness function

File: temp.urdf (robot description, URDF)
Before this commit: robot pepe, 6 links, 5 joints
Links:
- removed link 22
- removed link 43
- removed link 44
- removed link 45
- added link 42, mass 0.2973244783696758; collision cylinder length=0.36404158469510395 radius=0.5098763853987075; visual cylinder length=0.36404158469510395 radius=0.5098763853987075
- link 0: mass 0.0006823501410086211 -> 1.7777385015446838; geometry collision cylinder length=0.9415932321753037 radius=0.775224230565307; visual cylinder length=0.9415932321753037 radius=0.775224230565307
- link 21: mass 0.26933465574560406 -> 0.12530155718804586; geometry collision cylinder length=0.1660191363067025 radius=0.4901446004230555; visual cylinder length=0.1660191363067025 radius=0.4901446004230555
Joints:
- removed joint 22_to_0
- removed joint 43_to_0
- removed joint 44_to_0
- removed joint 45_to_0
- added joint 42_to_0: type fixed, parent 0, child 42, origin xyz=0.9582567832427751 0.4979230296828998 0.2894545214427092 rpy=17.20238513832142 0.05475282596471254 1.8604984463277343, axis 0 0 1, limit lower=1 upper=0 effort=1 velocity=1
- joint 21_to_0: axis 1 0 0 -> 0 1 0; origin xyz=0.36975590798791225 0.47915007546457045 0.6594773033465711 rpy=11.972928142491938 3.73866052011883 2.420214871450359 -> xyz=0.29605574810091106 0.2151043458850822 0.7690789732258686 rpy=2.9181664793893676 3.5831561125131293 1.1521662774467147

File: test.urdf (robot description, URDF)
Before this commit: robot pepe, 21 links, 20 joints
Links:
- removed link 412
- removed link 42
- removed link 47
- removed link 610
- removed link 611
- removed link 613
- removed link 614
- removed link 615
- removed link 616
- removed link 63
- removed link 64
- removed link 66
- removed link 68
- removed link 69
- removed link 817
- removed link 818
- removed link 819
- removed link 820
- added link 22, mass 0.04895270197432238; collision cylinder length=0.23860592413109016 radius=0.2555481766225518; visual cylinder length=0.23860592413109016 radius=0.2555481766225518
- added link 43, mass 2.48296840074274; collision cylinder length=0.9226564258106021 radius=0.9255303284190362; visual cylinder length=0.9226564258106021 radius=0.9255303284190362
- added link 44, mass 2.48296840074274; collision cylinder length=0.9226564258106021 radius=0.9255303284190362; visual cylinder length=0.9226564258106021 radius=0.9255303284190362
- added link 86, mass 0.3279253542393508; collision cylinder length=0.22961061582636 radius=0.6742432077970717; visual cylinder length=0.22961061582636 radius=0.6742432077970717
- link 0: mass 0.48167678407889525 -> 0.19758221768594314; geometry collision cylinder length=0.3069804814635626 radius=0.4526302863442113; visual cylinder length=0.3069804814635626 radius=0.4526302863442113
- link 21: mass 0.3517009485578119 -> 0.04895270197432238; geometry collision cylinder length=0.23860592413109016 radius=0.2555481766225518; visual cylinder length=0.23860592413109016 radius=0.2555481766225518
- link 65: mass 0.22329004334489153 -> 0.14295825448783808; geometry collision cylinder length=0.1339008708936278 radius=0.5829589593116505; visual cylinder length=0.1339008708936278 radius=0.5829589593116505
Joints:
- removed joint 412_to_0
- removed joint 42_to_0
- removed joint 47_to_0
- removed joint 610_to_47
- removed joint 611_to_47
- removed joint 613_to_412
- removed joint 614_to_412
- removed joint 615_to_412
- removed joint 616_to_412
- removed joint 63_to_42
- removed joint 64_to_42
- removed joint 65_to_42
- removed joint 66_to_42
- removed joint 68_to_47
- removed joint 69_to_47
- removed joint 817_to_0
- removed joint 818_to_0
- removed joint 819_to_0
- removed joint 820_to_0
- added joint 22_to_0: type fixed, parent 0, child 22, origin xyz=0.24827274272018662 0.04742562379229731 0.05586864175595618 rpy=15.775250092108013 2.2279177502046497 6.134383664500356, axis 1 0 0, limit lower=1 upper=0 effort=1 velocity=1
- added joint 43_to_0: type fixed, parent 0, child 43, origin xyz=0.8827948022963117 0.5175177817374326 0.24780670372275448 rpy=7.34216439299922 3.324163712810731 0.3113153484387992, axis 0 0 1, limit lower=1 upper=0 effort=1 velocity=1
- added joint 44_to_0: type fixed, parent 0, child 44, origin xyz=0.8827948022963117 0.5175177817374326 0.24780670372275448 rpy=9.177705491249025 3.324163712810731 0.3113153484387992, axis 0 0 1, limit lower=1 upper=0 effort=1 velocity=1
- added joint 65_to_0: type revolute, parent 0, child 65, origin xyz=0.6401690369091297 0.867020009642189 0.06460719749196986 rpy=20.83582780118447 2.239158249732535 5.258110035675699, axis 0 0 1, limit lower=1 upper=0 effort=1 velocity=1
- added joint 86_to_65: type fixed, parent 65, child 86, origin xyz=0.10726730001765317 0.3562572540806469 0.0928288310996348 rpy=6.852780235179486 0.6034117056732899 3.0858252787530227, axis 1 0 0, limit lower=1 upper=0 effort=1 velocity=1
- joint 21_to_0: axis 0 0 1 -> 1 0 0; origin xyz=0.4049974900486498 0.29998392026674536 0.7898189595844443 rpy=2.882601938893883 3.9758946769399803 1.974408129937515 -> xyz=0.24827274272018662 0.04742562379229731 0.05586864175595618 rpy=10.516833394738676 2.2279177502046497 6.134383664500356
