Commit message: edited

File: temp0.urdf (robot description, URDF)
Before this commit: robot pepe, 16 links, 15 joints
Links:
- removed link 211
- removed link 26
- removed link 410
- removed link 412
- removed link 413
- removed link 414
- removed link 415
- removed link 42
- removed link 43
- removed link 47
- removed link 48
- removed link 49
- added link 22, mass 0.39715143187843216; collision cylinder length=0.13012545824810529 radius=0.9856483382052503; visual cylinder length=0.13012545824810529 radius=0.9856483382052503
- added link 23, mass 0.39715143187843216; collision cylinder length=0.13012545824810529 radius=0.9856483382052503; visual cylinder length=0.13012545824810529 radius=0.9856483382052503
- link 0: mass 0.43425665619273307 -> 0.15005043868287074; geometry collision cylinder length=0.44125991091706085 radius=0.32900042721452183; visual cylinder length=0.44125991091706085 radius=0.32900042721452183
- link 21: mass 2.666863169662406 -> 0.39715143187843216; geometry collision cylinder length=0.13012545824810529 radius=0.9856483382052503; visual cylinder length=0.13012545824810529 radius=0.9856483382052503
- link 44: mass 1.1866796568520674 -> 1.0800840294395826; geometry collision cylinder length=0.8695597391725144 radius=0.62878782509659; visual cylinder length=0.8695597391725144 radius=0.62878782509659
- link 45: mass 1.1866796568520674 -> 1.0800840294395826; geometry collision cylinder length=0.8695597391725144 radius=0.62878782509659; visual cylinder length=0.8695597391725144 radius=0.62878782509659
Joints:
- removed joint 211_to_0
- removed joint 26_to_0
- removed joint 410_to_26
- removed joint 412_to_211
- removed joint 413_to_211
- removed joint 414_to_211
- removed joint 415_to_211
- removed joint 42_to_21
- removed joint 43_to_21
- removed joint 44_to_21
- removed joint 45_to_21
- removed joint 47_to_26
- removed joint 48_to_26
- removed joint 49_to_26
- added joint 22_to_0: type revolute, parent 0, child 22, origin xyz=0.1110815887884623 0.08608464780718161 0.7552012316289255 rpy=13.791066944469044 5.669523382641658 4.488867568695215, axis 0 0 1, limit lower=1 upper=0 effort=1 velocity=1
- added joint 23_to_0: type revolute, parent 0, child 23, origin xyz=0.1110815887884623 0.08608464780718161 0.7552012316289255 rpy=18.38808925929206 5.669523382641658 4.488867568695215, axis 0 0 1, limit lower=1 upper=0 effort=1 velocity=1
- added joint 44_to_0: type revolute, parent 0, child 44, origin xyz=0.7171169661827387 0.5265312303077535 0.0735165611367804 rpy=23.389764404049387 5.4319023001719104 3.0851368318284798, axis 1 0 0, limit lower=1 upper=0 effort=1 velocity=1
- added joint 45_to_0: type revolute, parent 0, child 45, origin xyz=0.7171169661827387 0.5265312303077535 0.0735165611367804 rpy=28.067717284859267 5.4319023001719104 3.0851368318284798, axis 1 0 0, limit lower=1 upper=0 effort=1 velocity=1
- joint 21_to_0: axis 0 1 0 -> 0 0 1; origin xyz=0.33784389938984294 0.7141984006028903 0.10117026484922664 rpy=12.12687725408024 0.3870160899212371 1.1109198743296802 -> xyz=0.1110815887884623 0.08608464780718161 0.7552012316289255 rpy=9.19404462964603 5.669523382641658 4.488867568695215

Commit message: roulette wheel selection

File: temp0.urdf (robot description, URDF)
Before this commit: robot pepe, 6 links, 5 joints
Links:
- removed link 22
- removed link 23
- removed link 44
- added link 24, mass 0.0025631275612023915; collision cylinder length=0.2991611899273102 radius=0.05222248670013241; visual cylinder length=0.2991611899273102 radius=0.05222248670013241
- added link 27, mass 0.0025631275612023915; collision cylinder length=0.2991611899273102 radius=0.05222248670013241; visual cylinder length=0.2991611899273102 radius=0.05222248670013241
- added link 42, mass 0.3885546329230645; collision cylinder length=0.27153568304292486 radius=0.6748972443308874; visual cylinder length=0.27153568304292486 radius=0.6748972443308874
- added link 43, mass 0.3885546329230645; collision cylinder length=0.27153568304292486 radius=0.6748972443308874; visual cylinder length=0.27153568304292486 radius=0.6748972443308874
- added link 46, mass 0.3885546329230645; collision cylinder length=0.27153568304292486 radius=0.6748972443308874; visual cylinder length=0.27153568304292486 radius=0.6748972443308874
- added link 48, mass 0.3885546329230645; collision cylinder length=0.27153568304292486 radius=0.6748972443308874; visual cylinder length=0.27153568304292486 radius=0.6748972443308874
- added link 49, mass 0.3885546329230645; collision cylinder length=0.27153568304292486 radius=0.6748972443308874; visual cylinder length=0.27153568304292486 radius=0.6748972443308874
- link 0: mass 0.15005043868287074 -> 0.1203356223649135; geometry collision cylinder length=0.3474069374356369 radius=0.33204957179699046; visual cylinder length=0.3474069374356369 radius=0.33204957179699046
- link 21: mass 0.39715143187843216 -> 0.0025631275612023915; geometry collision cylinder length=0.2991611899273102 radius=0.05222248670013241; visual cylinder length=0.2991611899273102 radius=0.05222248670013241
- link 45: mass 1.0800840294395826 -> 0.3885546329230645; geometry collision cylinder length=0.27153568304292486 radius=0.6748972443308874; visual cylinder length=0.27153568304292486 radius=0.6748972443308874
Joints:
- removed joint 22_to_0
- removed joint 23_to_0
- removed joint 44_to_0
- removed joint 45_to_0
- added joint 24_to_0: type revolute, parent 0, child 24, origin xyz=0.38735189703546813 0.36606842116948957 0.08090521909868242 rpy=11.157907987977971 4.063342342129231 6.060469224452089, axis 0 1 0, limit lower=1 upper=0 effort=1 velocity=1
- added joint 27_to_0: type revolute, parent 0, child 27, origin xyz=0.38735189703546813 0.36606842116948957 0.08090521909868242 rpy=14.877210650637295 4.063342342129231 6.060469224452089, axis 0 1 0, limit lower=1 upper=0 effort=1 velocity=1
- added joint 42_to_21: type revolute, parent 21, child 42, origin xyz=0.6498149244525386 0.9613505685216701 0.19499530593404524 rpy=7.49712228223505 5.6152602922292045 4.571884343995946, axis 1 0 0, limit lower=1 upper=0 effort=1 velocity=1
- added joint 43_to_21: type revolute, parent 21, child 43, origin xyz=0.6498149244525386 0.9613505685216701 0.19499530593404524 rpy=11.245683423352574 5.6152602922292045 4.571884343995946, axis 1 0 0, limit lower=1 upper=0 effort=1 velocity=1
- added joint 45_to_24: type revolute, parent 24, child 45, origin xyz=0.6498149244525386 0.9613505685216701 0.19499530593404524 rpy=7.49712228223505 5.6152602922292045 4.571884343995946, axis 1 0 0, limit lower=1 upper=0 effort=1 velocity=1
- added joint 46_to_24: type revolute, parent 24, child 46, origin xyz=0.6498149244525386 0.9613505685216701 0.19499530593404524 rpy=11.245683423352574 5.6152602922292045 4.571884343995946, axis 1 0 0, limit lower=1 upper=0 effort=1 velocity=1
- added joint 48_to_27: type revolute, parent 27, child 48, origin xyz=0.6498149244525386 0.9613505685216701 0.19499530593404524 rpy=7.49712228223505 5.6152602922292045 4.571884343995946, axis 1 0 0, limit lower=1 upper=0 effort=1 velocity=1
- added joint 49_to_27: type revolute, parent 27, child 49, origin xyz=0.6498149244525386 0.9613505685216701 0.19499530593404524 rpy=11.245683423352574 5.6152602922292045 4.571884343995946, axis 1 0 0, limit lower=1 upper=0 effort=1 velocity=1
- joint 21_to_0: axis 0 0 1 -> 0 1 0; origin xyz=0.1110815887884623 0.08608464780718161 0.7552012316289255 rpy=9.19404462964603 5.669523382641658 4.488867568695215 -> xyz=0.38735189703546813 0.36606842116948957 0.08090521909868242 rpy=7.4386053253186475 4.063342342129231 6.060469224452089

Commit message: simple evolution

File: temp0.urdf (robot description, URDF)
Before this commit: robot pepe, 10 links, 9 joints
Links:
- removed link 24
- removed link 27
- removed link 42
- removed link 43
- removed link 48
- removed link 49
- added link 22, mass 1.190145987856078; collision cylinder length=0.9137429897075929 radius=0.6438921835671327; visual cylinder length=0.9137429897075929 radius=0.6438921835671327
- added link 23, mass 1.190145987856078; collision cylinder length=0.9137429897075929 radius=0.6438921835671327; visual cylinder length=0.9137429897075929 radius=0.6438921835671327
- added link 44, mass 1.3803882913102732; collision cylinder length=0.8091630991505836 radius=0.7368984831101258; visual cylinder length=0.8091630991505836 radius=0.7368984831101258
- link 0: mass 0.1203356223649135 -> 0.09655615929846667; geometry collision cylinder length=0.8800497900486061 radius=0.18687940087076782; visual cylinder length=0.8800497900486061 radius=0.18687940087076782
- link 21: mass 0.0025631275612023915 -> 1.190145987856078; geometry collision cylinder length=0.9137429897075929 radius=0.6438921835671327; visual cylinder length=0.9137429897075929 radius=0.6438921835671327
- link 45: mass 0.3885546329230645 -> 1.3803882913102732; geometry collision cylinder length=0.8091630991505836 radius=0.7368984831101258; visual cylinder length=0.8091630991505836 radius=0.7368984831101258
- link 46: mass 0.3885546329230645 -> 1.3803882913102732; geometry collision cylinder length=0.8091630991505836 radius=0.7368984831101258; visual cylinder length=0.8091630991505836 radius=0.7368984831101258
Joints:
- removed joint 24_to_0
- removed joint 27_to_0
- removed joint 42_to_21
- removed joint 43_to_21
- removed joint 45_to_24
- removed joint 46_to_24
- removed joint 48_to_27
- removed joint 49_to_27
- added joint 22_to_0: type fixed, parent 0, child 22, origin xyz=0.25539511636069523 0.02552781582124597 0.9475054482956785 rpy=8.043514908196446 1.4486528267828158 3.4112814727526755, axis 0 0 1, limit lower=1 upper=0 effort=1 velocity=1
- added joint 23_to_0: type fixed, parent 0, child 23, origin xyz=0.25539511636069523 0.02552781582124597 0.9475054482956785 rpy=10.724686544261928 1.4486528267828158 3.4112814727526755, axis 0 0 1, limit lower=1 upper=0 effort=1 velocity=1
- added joint 44_to_0: type revolute, parent 0, child 44, origin xyz=0.3100571897034001 0.13606985150967332 0.29339288493107885 rpy=15.036341553898676 0.5132524082122799 5.464722297293214, axis 1 0 0, limit lower=1 upper=0 effort=1 velocity=1
- added joint 45_to_0: type revolute, parent 0, child 45, origin xyz=0.3100571897034001 0.13606985150967332 0.29339288493107885 rpy=18.04360986467841 0.5132524082122799 5.464722297293214, axis 1 0 0, limit lower=1 upper=0 effort=1 velocity=1
- added joint 46_to_0: type revolute, parent 0, child 46, origin xyz=0.3100571897034001 0.13606985150967332 0.29339288493107885 rpy=21.050878175458145 0.5132524082122799 5.464722297293214, axis 1 0 0, limit lower=1 upper=0 effort=1 velocity=1
- joint 21_to_0: axis 0 1 0 -> 0 0 1; origin xyz=0.38735189703546813 0.36606842116948957 0.08090521909868242 rpy=7.4386053253186475 4.063342342129231 6.060469224452089 -> xyz=0.25539511636069523 0.02552781582124597 0.9475054482956785 rpy=5.362343272130964 1.4486528267828158 3.4112814727526755; type revolute -> fixed

Commit message: tweaking the GA

File: temp0.urdf (robot description, URDF)
Before this commit: robot pepe, 7 links, 6 joints
Links:
- removed link 22
- removed link 23
- removed link 44
- removed link 46
- added link 28, mass 0.6426538132963756; collision cylinder length=0.9126648145056405 radius=0.47343237608486655; visual cylinder length=0.9126648145056405 radius=0.47343237608486655
- added link 412, mass 0.4507547137594424; collision cylinder length=0.20982994091259813 radius=0.8269161481953621; visual cylinder length=0.20982994091259813 radius=0.8269161481953621
- added link 42, mass 0.4507547137594424; collision cylinder length=0.20982994091259813 radius=0.8269161481953621; visual cylinder length=0.20982994091259813 radius=0.8269161481953621
- added link 49, mass 0.4507547137594424; collision cylinder length=0.20982994091259813 radius=0.8269161481953621; visual cylinder length=0.20982994091259813 radius=0.8269161481953621
- added link 610, mass 0.10849184608437856; collision cylinder length=0.8845853037265385 radius=0.1975849008266123; visual cylinder length=0.8845853037265385 radius=0.1975849008266123
- added link 611, mass 0.10849184608437856; collision cylinder length=0.8845853037265385 radius=0.1975849008266123; visual cylinder length=0.8845853037265385 radius=0.1975849008266123
- added link 613, mass 0.10849184608437856; collision cylinder length=0.8845853037265385 radius=0.1975849008266123; visual cylinder length=0.8845853037265385 radius=0.1975849008266123
- added link 614, mass 0.10849184608437856; collision cylinder length=0.8845853037265385 radius=0.1975849008266123; visual cylinder length=0.8845853037265385 radius=0.1975849008266123
- added link 63, mass 0.10849184608437856; collision cylinder length=0.8845853037265385 radius=0.1975849008266123; visual cylinder length=0.8845853037265385 radius=0.1975849008266123
- added link 64, mass 0.10849184608437856; collision cylinder length=0.8845853037265385 radius=0.1975849008266123; visual cylinder length=0.8845853037265385 radius=0.1975849008266123
- added link 66, mass 0.10849184608437856; collision cylinder length=0.8845853037265385 radius=0.1975849008266123; visual cylinder length=0.8845853037265385 radius=0.1975849008266123
- added link 67, mass 0.10849184608437856; collision cylinder length=0.8845853037265385 radius=0.1975849008266123; visual cylinder length=0.8845853037265385 radius=0.1975849008266123
- link 0: mass 0.09655615929846667 -> 0.07790804190274214; geometry collision cylinder length=0.9453461753062888 radius=0.16196484976351178; visual cylinder length=0.9453461753062888 radius=0.16196484976351178
- link 21: mass 1.190145987856078 -> 0.6426538132963756; geometry collision cylinder length=0.9126648145056405 radius=0.47343237608486655; visual cylinder length=0.9126648145056405 radius=0.47343237608486655
- link 45: mass 1.3803882913102732 -> 0.4507547137594424; geometry collision cylinder length=0.20982994091259813 radius=0.8269161481953621; visual cylinder length=0.20982994091259813 radius=0.8269161481953621
Joints:
- removed joint 22_to_0
- removed joint 23_to_0
- removed joint 44_to_0
- removed joint 45_to_0
- removed joint 46_to_0
- added joint 28_to_0: type revolute, parent 0, child 28, origin xyz=0.9706059983352722 0.2980307351955784 0.4687002655631931 rpy=1.9471333321366755 1.5246346562755937 2.609385264902831, axis 1 0 0, limit lower=1 upper=0 effort=1 velocity=1
- added joint 412_to_28: type revolute, parent 28, child 412, origin xyz=0.779911147843065 0.8005702482773761 0.8766504826284565 rpy=18.70925492950711 5.543990825183449 2.5534880103461295, axis 0 0 1, limit lower=1 upper=0 effort=1 velocity=1
- added joint 42_to_21: type revolute, parent 21, child 42, origin xyz=0.779911147843065 0.8005702482773761 0.8766504826284565 rpy=12.472836619671408 5.543990825183449 2.5534880103461295, axis 0 0 1, limit lower=1 upper=0 effort=1 velocity=1
- added joint 45_to_21: type revolute, parent 21, child 45, origin xyz=0.779911147843065 0.8005702482773761 0.8766504826284565 rpy=18.70925492950711 5.543990825183449 2.5534880103461295, axis 0 0 1, limit lower=1 upper=0 effort=1 velocity=1
- added joint 49_to_28: type revolute, parent 28, child 49, origin xyz=0.779911147843065 0.8005702482773761 0.8766504826284565 rpy=12.472836619671408 5.543990825183449 2.5534880103461295, axis 0 0 1, limit lower=1 upper=0 effort=1 velocity=1
- added joint 610_to_49: type fixed, parent 49, child 610, origin xyz=0.6866744144153338 0.7734064437958295 0.9403078155385293 rpy=6.299360428325358 1.7510110390331635 6.227357477000398, axis 1 0 0, limit lower=1 upper=0 effort=1 velocity=1
- added joint 611_to_49: type fixed, parent 49, child 611, origin xyz=0.6866744144153338 0.7734064437958295 0.9403078155385293 rpy=9.449040642488038 1.7510110390331635 6.227357477000398, axis 1 0 0, limit lower=1 upper=0 effort=1 velocity=1
- added joint 613_to_412: type fixed, parent 412, child 613, origin xyz=0.6866744144153338 0.7734064437958295 0.9403078155385293 rpy=6.299360428325358 1.7510110390331635 6.227357477000398, axis 1 0 0, limit lower=1 upper=0 effort=1 velocity=1
- added joint 614_to_412: type fixed, parent 412, child 614, origin xyz=0.6866744144153338 0.7734064437958295 0.9403078155385293 rpy=9.449040642488038 1.7510110390331635 6.227357477000398, axis 1 0 0, limit lower=1 upper=0 effort=1 velocity=1
- added joint 63_to_42: type fixed, parent 42, child 63, origin xyz=0.6866744144153338 0.7734064437958295 0.9403078155385293 rpy=6.299360428325358 1.7510110390331635 6.227357477000398, axis 1 0 0, limit lower=1 upper=0 effort=1 velocity=1
- added joint 64_to_42: type fixed, parent 42, child 64, origin xyz=0.6866744144153338 0.7734064437958295 0.9403078155385293 rpy=9.449040642488038 1.7510110390331635 6.227357477000398, axis 1 0 0, limit lower=1 upper=0 effort=1 velocity=1
- added joint 66_to_45: type fixed, parent 45, child 66, origin xyz=0.6866744144153338 0.7734064437958295 0.9403078155385293 rpy=6.299360428325358 1.7510110390331635 6.227357477000398, axis 1 0 0, limit lower=1 upper=0 effort=1 velocity=1
- added joint 67_to_45: type fixed, parent 45, child 67, origin xyz=0.6866744144153338 0.7734064437958295 0.9403078155385293 rpy=9.449040642488038 1.7510110390331635 6.227357477000398, axis 1 0 0, limit lower=1 upper=0 effort=1 velocity=1
- joint 21_to_0: axis 0 0 1 -> 1 0 0; origin xyz=0.25539511636069523 0.02552781582124597 0.9475054482956785 rpy=5.362343272130964 1.4486528267828158 3.4112814727526755 -> xyz=0.9706059983352722 0.2980307351955784 0.4687002655631931 rpy=1.298088888091117 1.5246346562755937 2.609385264902831; type fixed -> revolute
