Commit message: saving and viewing fittest

File: temp0.urdf (robot description, URDF)
Before this commit: robot pepe, 15 links, 14 joints
Links:
- removed link 28
- removed link 412
- removed link 42
- removed link 45
- removed link 49
- removed link 610
- removed link 611
- removed link 613
- removed link 63
- removed link 66
- removed link 67
- added link 22, mass 0.0019605540409321632; collision cylinder length=0.000734617363635337 radius=0.9216878826634727; visual cylinder length=0.000734617363635337 radius=0.9216878826634727
- added link 413, mass 1.1662843146456345; collision cylinder length=0.4352275761186666 radius=0.9235684291979013; visual cylinder length=0.4352275761186666 radius=0.9235684291979013
- added link 418, mass 1.1662843146456345; collision cylinder length=0.4352275761186666 radius=0.9235684291979013; visual cylinder length=0.4352275761186666 radius=0.9235684291979013
- added link 43, mass 1.1662843146456345; collision cylinder length=0.4352275761186666 radius=0.9235684291979013; visual cylinder length=0.4352275761186666 radius=0.9235684291979013
- added link 48, mass 1.1662843146456345; collision cylinder length=0.4352275761186666 radius=0.9235684291979013; visual cylinder length=0.4352275761186666 radius=0.9235684291979013
- added link 619, mass 0.424927211067474; collision cylinder length=0.5189468049023803 radius=0.5105295844709402; visual cylinder length=0.5189468049023803 radius=0.5105295844709402
- added link 69, mass 0.424927211067474; collision cylinder length=0.5189468049023803 radius=0.5105295844709402; visual cylinder length=0.5189468049023803 radius=0.5105295844709402
- added link 810, mass 0.5496541579025842; collision cylinder length=0.5518670968100813 radius=0.5630572717876117; visual cylinder length=0.5518670968100813 radius=0.5630572717876117
- added link 811, mass 0.5496541579025842; collision cylinder length=0.5518670968100813 radius=0.5630572717876117; visual cylinder length=0.5518670968100813 radius=0.5630572717876117
- added link 812, mass 0.5496541579025842; collision cylinder length=0.5518670968100813 radius=0.5630572717876117; visual cylinder length=0.5518670968100813 radius=0.5630572717876117
- added link 815, mass 0.5496541579025842; collision cylinder length=0.5518670968100813 radius=0.5630572717876117; visual cylinder length=0.5518670968100813 radius=0.5630572717876117
- added link 816, mass 0.5496541579025842; collision cylinder length=0.5518670968100813 radius=0.5630572717876117; visual cylinder length=0.5518670968100813 radius=0.5630572717876117
- added link 817, mass 0.5496541579025842; collision cylinder length=0.5518670968100813 radius=0.5630572717876117; visual cylinder length=0.5518670968100813 radius=0.5630572717876117
- added link 820, mass 0.5496541579025842; collision cylinder length=0.5518670968100813 radius=0.5630572717876117; visual cylinder length=0.5518670968100813 radius=0.5630572717876117
- added link 821, mass 0.5496541579025842; collision cylinder length=0.5518670968100813 radius=0.5630572717876117; visual cylinder length=0.5518670968100813 radius=0.5630572717876117
- added link 822, mass 0.5496541579025842; collision cylinder length=0.5518670968100813 radius=0.5630572717876117; visual cylinder length=0.5518670968100813 radius=0.5630572717876117
- added link 85, mass 0.5496541579025842; collision cylinder length=0.5518670968100813 radius=0.5630572717876117; visual cylinder length=0.5518670968100813 radius=0.5630572717876117
- added link 86, mass 0.5496541579025842; collision cylinder length=0.5518670968100813 radius=0.5630572717876117; visual cylinder length=0.5518670968100813 radius=0.5630572717876117
- added link 87, mass 0.5496541579025842; collision cylinder length=0.5518670968100813 radius=0.5630572717876117; visual cylinder length=0.5518670968100813 radius=0.5630572717876117
- link 0: mass 0.07790804190274214 -> 0.11307014476675485; geometry collision cylinder length=0.721742419142738 radius=0.22330987182540718; visual cylinder length=0.721742419142738 radius=0.22330987182540718
- link 21: mass 0.6426538132963756 -> 0.0019605540409321632; geometry collision cylinder length=0.000734617363635337 radius=0.9216878826634727; visual cylinder length=0.000734617363635337 radius=0.9216878826634727
- link 614: mass 0.10849184608437856 -> 0.424927211067474; geometry collision cylinder length=0.5189468049023803 radius=0.5105295844709402; visual cylinder length=0.5189468049023803 radius=0.5105295844709402
- link 64: mass 0.10849184608437856 -> 0.424927211067474; geometry collision cylinder length=0.5189468049023803 radius=0.5105295844709402; visual cylinder length=0.5189468049023803 radius=0.5105295844709402
Joints:
- removed joint 28_to_0
- removed joint 412_to_28
- removed joint 42_to_21
- removed joint 45_to_21
- removed joint 49_to_28
- removed joint 610_to_49
- removed joint 611_to_49
- removed joint 613_to_412
- removed joint 614_to_412
- removed joint 63_to_42
- removed joint 64_to_42
- removed joint 66_to_45
- removed joint 67_to_45
- added joint 22_to_0: type revolute, parent 0, child 22, origin xyz=0.32499494564946707 0.51097141962273 0.8391477240248747 rpy=4.907758408387075 0.9123943742054137 2.44217369908531, axis 0 1 0, limit lower=1 upper=0 effort=1 velocity=1
- added joint 413_to_0: type revolute, parent 0, child 413, origin xyz=0.8052657009323001 0.7459523450254745 0.01938024093207158 rpy=3.0252564405625044 3.5627435229866906 4.650508314697615, axis 0 1 0, limit lower=1 upper=0 effort=1 velocity=1
- added joint 418_to_0: type revolute, parent 0, child 418, origin xyz=0.8052657009323001 0.7459523450254745 0.01938024093207158 rpy=3.5294658473229217 3.5627435229866906 4.650508314697615, axis 0 1 0, limit lower=1 upper=0 effort=1 velocity=1
- added joint 43_to_0: type revolute, parent 0, child 43, origin xyz=0.8052657009323001 0.7459523450254745 0.01938024093207158 rpy=2.0168376270416695 3.5627435229866906 4.650508314697615, axis 0 1 0, limit lower=1 upper=0 effort=1 velocity=1
- added joint 48_to_0: type revolute, parent 0, child 48, origin xyz=0.8052657009323001 0.7459523450254745 0.01938024093207158 rpy=2.5210470338020867 3.5627435229866906 4.650508314697615, axis 0 1 0, limit lower=1 upper=0 effort=1 velocity=1
- added joint 614_to_413: type fixed, parent 413, child 614, origin xyz=0.5649444572458518 0.2111526948347282 0.1423473639036058 rpy=8.323420897472007 5.641960473356935 3.1007381027058014, axis 0 0 1, limit lower=1 upper=0 effort=1 velocity=1
- added joint 619_to_418: type fixed, parent 418, child 619, origin xyz=0.5649444572458518 0.2111526948347282 0.1423473639036058 rpy=8.323420897472007 5.641960473356935 3.1007381027058014, axis 0 0 1, limit lower=1 upper=0 effort=1 velocity=1
- added joint 64_to_43: type fixed, parent 43, child 64, origin xyz=0.5649444572458518 0.2111526948347282 0.1423473639036058 rpy=8.323420897472007 5.641960473356935 3.1007381027058014, axis 0 0 1, limit lower=1 upper=0 effort=1 velocity=1
- added joint 69_to_48: type fixed, parent 48, child 69, origin xyz=0.5649444572458518 0.2111526948347282 0.1423473639036058 rpy=8.323420897472007 5.641960473356935 3.1007381027058014, axis 0 0 1, limit lower=1 upper=0 effort=1 velocity=1
- added joint 810_to_69: type revolute, parent 69, child 810, origin xyz=0.3646892100973431 0.4877004974643625 0.8009978672506617 rpy=3.731045533978844 3.9203898011542293 5.540014039112312, axis 1 0 0, limit lower=1 upper=0 effort=1 velocity=1
- added joint 811_to_69: type revolute, parent 69, child 811, origin xyz=0.3646892100973431 0.4877004974643625 0.8009978672506617 rpy=5.596568300968267 3.9203898011542293 5.540014039112312, axis 1 0 0, limit lower=1 upper=0 effort=1 velocity=1
- added joint 812_to_69: type revolute, parent 69, child 812, origin xyz=0.3646892100973431 0.4877004974643625 0.8009978672506617 rpy=7.462091067957688 3.9203898011542293 5.540014039112312, axis 1 0 0, limit lower=1 upper=0 effort=1 velocity=1
- added joint 815_to_614: type revolute, parent 614, child 815, origin xyz=0.3646892100973431 0.4877004974643625 0.8009978672506617 rpy=3.731045533978844 3.9203898011542293 5.540014039112312, axis 1 0 0, limit lower=1 upper=0 effort=1 velocity=1
- added joint 816_to_614: type revolute, parent 614, child 816, origin xyz=0.3646892100973431 0.4877004974643625 0.8009978672506617 rpy=5.596568300968267 3.9203898011542293 5.540014039112312, axis 1 0 0, limit lower=1 upper=0 effort=1 velocity=1
- added joint 817_to_614: type revolute, parent 614, child 817, origin xyz=0.3646892100973431 0.4877004974643625 0.8009978672506617 rpy=7.462091067957688 3.9203898011542293 5.540014039112312, axis 1 0 0, limit lower=1 upper=0 effort=1 velocity=1
- added joint 820_to_619: type revolute, parent 619, child 820, origin xyz=0.3646892100973431 0.4877004974643625 0.8009978672506617 rpy=3.731045533978844 3.9203898011542293 5.540014039112312, axis 1 0 0, limit lower=1 upper=0 effort=1 velocity=1
- added joint 821_to_619: type revolute, parent 619, child 821, origin xyz=0.3646892100973431 0.4877004974643625 0.8009978672506617 rpy=5.596568300968267 3.9203898011542293 5.540014039112312, axis 1 0 0, limit lower=1 upper=0 effort=1 velocity=1
- added joint 822_to_619: type revolute, parent 619, child 822, origin xyz=0.3646892100973431 0.4877004974643625 0.8009978672506617 rpy=7.462091067957688 3.9203898011542293 5.540014039112312, axis 1 0 0, limit lower=1 upper=0 effort=1 velocity=1
- added joint 85_to_64: type revolute, parent 64, child 85, origin xyz=0.3646892100973431 0.4877004974643625 0.8009978672506617 rpy=3.731045533978844 3.9203898011542293 5.540014039112312, axis 1 0 0, limit lower=1 upper=0 effort=1 velocity=1
- added joint 86_to_64: type revolute, parent 64, child 86, origin xyz=0.3646892100973431 0.4877004974643625 0.8009978672506617 rpy=5.596568300968267 3.9203898011542293 5.540014039112312, axis 1 0 0, limit lower=1 upper=0 effort=1 velocity=1
- added joint 87_to_64: type revolute, parent 64, child 87, origin xyz=0.3646892100973431 0.4877004974643625 0.8009978672506617 rpy=7.462091067957688 3.9203898011542293 5.540014039112312, axis 1 0 0, limit lower=1 upper=0 effort=1 velocity=1
- joint 21_to_0: axis 1 0 0 -> 0 1 0; origin xyz=0.9706059983352722 0.2980307351955784 0.4687002655631931 rpy=1.298088888091117 1.5246346562755937 2.609385264902831 -> xyz=0.32499494564946707 0.51097141962273 0.8391477240248747 rpy=3.2718389389247164 0.9123943742054137 2.44217369908531

File: test.urdf (robot description, URDF)
Before this commit: robot pepe, 7 links, 6 joints
Links:
- removed link 22
- removed link 43
- removed link 44
- removed link 65
- removed link 86
- added link 42, mass 0.26269059710040277; collision cylinder length=0.2315967112959374 radius=0.6008708469982534; visual cylinder length=0.2315967112959374 radius=0.6008708469982534
- link 0: mass 0.19758221768594314 -> 0.037111354572574445; geometry collision cylinder length=0.25950162733891324 radius=0.21335775063027462; visual cylinder length=0.25950162733891324 radius=0.21335775063027462
- link 21: mass 0.04895270197432238 -> 0.0013450359108385973; geometry collision cylinder length=0.12842367253876308 radius=0.057739026974342744; visual cylinder length=0.12842367253876308 radius=0.057739026974342744
Joints:
- removed joint 22_to_0
- removed joint 43_to_0
- removed joint 44_to_0
- removed joint 65_to_0
- removed joint 86_to_65
- added joint 42_to_21: type revolute, parent 21, child 42, origin xyz=0.755944140376686 0.8709923196478481 0.26541584884625624 rpy=5.544826369359781 5.273315625365528 3.7493644256969954, axis 0 0 1, limit lower=1 upper=0 effort=1 velocity=1
- joint 21_to_0: axis 1 0 0 -> 0 1 0; origin xyz=0.24827274272018662 0.04742562379229731 0.05586864175595618 rpy=10.516833394738676 2.2279177502046497 6.134383664500356 -> xyz=0.644031000195063 0.09318712703529886 0.3682030709216344 rpy=7.518330377270403 6.189052547967725 6.244769511975179; type fixed -> revolute
